Commit message: feat: add broken sim

File: guide_robot_description/urdf/guide_robot.ros2_control.xacro (robot description, xacro)
@@ -1,35 +1,47 @@
 <?xml version="1.0"?>
 <!-- =========================================================================
-     ros2_control интерфейс для Guide robot.
-     Аргумент use_sim переключает на mock-железо для проверки без робота.
+     ros2_control interface for Guide robot.
+     Three hardware backends, priority top to bottom:
+       use_sim=true           -> Gazebo Classic (gazebo_ros2_control)
+       use_mock_hardware=true -> mock_components stub for stack testing
+       otherwise              -> real Dynamixel driver
+     IMPORTANT: comments MUST stay ASCII-only (see note in guide_robot.urdf.xacro).
      ========================================================================= -->
 <robot xmlns:xacro="http://www.ros.org/wiki/xacro">
+  <xacro:arg name="use_sim"           default="false"/>
   <xacro:arg name="use_mock_hardware" default="false"/>
   <ros2_control name="GuideRobotSystem" type="system">
     <hardware>
-      <xacro:if value="$(arg use_mock_hardware)">
-        <!-- Заглушка для запуска стека без реального робота -->
-        <plugin>mock_components/GenericSystem</plugin>
-        <param name="calculate_dynamics">true</param>
+      <xacro:if value="$(arg use_sim)">
+        <!-- Gazebo Classic: simulated hardware via gazebo_ros2_control.
+             Drives the same velocity interfaces as the real base. -->
+        <plugin>gazebo_ros2_control/GazeboSystem</plugin>
       </xacro:if>
-      <xacro:unless value="$(arg use_mock_hardware)">
-        <!-- Реальный драйвер Dynamixel-базы Guide Robot -->
-        <plugin>guide_robot_hardware/GuideRobotSystem</plugin>
-        <param name="serial_port">COM7</param>  <!-- TO-DO -->
-        <param name="baud_rate">115200</param>
-        <param name="left_wheel_id">46</param>           <!-- 0x2E -->
-        <param name="right_wheel_id">47</param>          <!-- 0x2F -->
-        <param name="ticks_per_rev">262144</param>       <!-- 512*8*64 -->
-        <param name="left_sign">-1</param>               <!-- LeftReverse -->
-        <param name="right_sign">1</param>               <!-- RightReverse -->
-        <param name="swap_drives">1</param>              <!-- FURO_SWAP_DRIVES -->
-        <param name="speed_coefficient">0.014</param>    <!-- м/с -->
-        <param name="cmd_timeout">0.3</param>            <!-- watchdog, сек -->
+      <xacro:unless value="$(arg use_sim)">
+        <xacro:if value="$(arg use_mock_hardware)">
+          <!-- Stub for running the stack without real hardware -->
+          <plugin>mock_components/GenericSystem</plugin>
+          <param name="calculate_dynamics">true</param>
+        </xacro:if>
+        <xacro:unless value="$(arg use_mock_hardware)">
+          <!-- Real Dynamixel base driver -->
+          <plugin>guide_robot_hardware/GuideRobotSystem</plugin>
+          <param name="serial_port">COM7</param>            <!-- TO-DO -->
+          <param name="baud_rate">115200</param>
+          <param name="left_wheel_id">46</param>            <!-- 0x2E -->
+          <param name="right_wheel_id">47</param>           <!-- 0x2F -->
+          <param name="ticks_per_rev">262144</param>        <!-- 512*8*64 -->
+          <param name="left_sign">-1</param>                <!-- LeftReverse -->
+          <param name="right_sign">1</param>                <!-- RightReverse -->
+          <param name="swap_drives">1</param>               <!-- FURO_SWAP_DRIVES -->
+          <param name="speed_coefficient">0.014</param>     <!-- m/s -->
+          <param name="cmd_timeout">0.3</param>             <!-- watchdog, sec -->
+        </xacro:unless>
       </xacro:unless>
     </hardware>
-    <!-- Левое колесо -->
+    <!-- Left wheel -->
     <joint name="left_wheel_joint">
       <command_interface name="velocity">
-        <param name="min">-6.98</param>   <!-- рад/с, ~= 0.3 м/с / 0.075 * запас -->
+        <param name="min">-6.98</param>   <!-- rad/s -->
         <param name="max">6.98</param>
       </command_interface>
@@ -37,5 +49,5 @@
       <state_interface name="velocity"/>
     </joint>
-    <!-- Правое колесо -->
+    <!-- Right wheel -->
     <joint name="right_wheel_joint">
       <command_interface name="velocity">

File: guide_robot_description/urdf/guide_robot.urdf.xacro (robot description, xacro)
@@ -1,29 +1,39 @@
 <?xml version="1.0"?>
 <!-- =========================================================================
-     Guide robot — основное описание робота.
-     Геометрия из RobotSetting.xml. Меши пока заменены примитивами
-     (цилиндр корпуса + цилиндры колёс) — этого достаточно для costmap и TF.
-     Крепления лидаров и соединительый профиль — реальные меши.
+     Guide robot - main robot description.
+     Geometry from RobotSetting.xml. Meshes are replaced by primitives for now
+     (body cylinder + wheel cylinders) - enough for costmap and TF.
+     Lidar mounts and connecting profile use real meshes.
+     Rear casters are a real part of the robot (top-heavy chassis support).
+     IMPORTANT: comments MUST stay ASCII-only. Non-ASCII characters break
+     gazebo_ros2_control, which passes robot_description as a CLI parameter
+     and truncates the buffer mid multi-byte sequence.
      ========================================================================= -->
 <robot xmlns:xacro="http://www.ros.org/wiki/xacro" name="guide_robot">
-  <!-- ===================== Параметры (из robot_params.yaml) ============== -->
-  <xacro:property name="wheel_separation" value="0.347"/>   <!-- WheelBase -->
-  <xacro:property name="wheel_radius"     value="0.075"/>    <!-- WheelDiameter/2 TO-DO -->
+  <!-- Simulation flag: enables gazebo plugins and switches hardware backend -->
+  <xacro:arg name="use_sim" default="false"/>
+  <!-- ===================== Parameters (from robot_params.yaml) =========== -->
+  <xacro:property name="wheel_separation" value="0.338"/>   <!-- WheelBase -->
+  <xacro:property name="wheel_radius"     value="0.075"/>    <!-- WheelDiameter/2 -->
   <xacro:property name="wheel_width"      value="0.048"/>    <!-- WheelWidth -->
-  <!-- Габариты корпуса — грубая оценка top-heavy шасси -->
+  <!-- Body dimensions - rough estimate of top-heavy chassis -->
   <xacro:property name="body_radius" value="0.31"/>
   <xacro:property name="body_height" value="1.62"/>
-  <xacro:property name="body_z"      value="0.675"/>          <!-- центр корпуса по Z-->
-  <!-- Клиренс: ось колёс над полом = wheel_radius -->
+  <xacro:property name="body_z"      value="0.885"/>         <!-- body center Z -->
+  <!-- Ground clearance: wheel axle height above floor = wheel_radius -->
   <xacro:property name="base_z" value="${wheel_radius}"/>
-  <!-- Крепления лидаров + соединительная палка (2020 экструзия) -->
+  <!-- Rear casters (real support) -->
+  <xacro:property name="caster_radius" value="${base_z}"/>   <!-- = wheel_radius, keeps robot level -->
+  <xacro:property name="caster_x"      value="-0.3"/>       <!-- behind base center, ~20 cm -->
+  <xacro:property name="caster_y"      value="0.12"/>        <!-- lateral spacing -->
+  <!-- Lidar mounts + connecting bar (2020 extrusion) -->
   <xacro:property name="lidar_mount_mesh" value="package://guide_robot_description/meshes/lidars_mount.stl"/>
   <xacro:property name="lidar_bar_mesh"   value="package://guide_robot_description/meshes/al_profile.stl"/>
-  <!-- TO-DO: если меши экспортированы из CAD в мм — нужен scale 0.001 0.001 0.001.
-       Проверить в RViz: огромная/крошечная модель = неверный scale. -->
+  <!-- TO-DO: if meshes were exported from CAD in mm, scale 0.001 is required.
+       Check in RViz: huge or tiny model means wrong scale. -->
   <xacro:property name="mesh_scale" value="0.001 0.001 0.001"/>
-  <xacro:property name="lidar_y_offset" value="0.258"/>       <!-- было в laser_joint_left/right -->
+  <xacro:property name="lidar_y_offset" value="0.258"/>      <!-- from laser_joint_left/right -->
   <xacro:property name="lidar_z" value="0.4"/>
-  <!-- ===================== Материалы для RViz ============================ -->
+  <!-- ===================== RViz materials =============================== -->
   <material name="grey"><color rgba="0.4 0.4 0.45 1.0"/></material>
   <material name="dark"><color rgba="0.15 0.15 0.15 1.0"/></material>
@@ -32,13 +42,13 @@
   <link name="base_footprint"/>
   <link name="base_link">
-    <!-- <visual>
-      <origin xyz="0 0 ${body_z - base_z}" rpy="0 0 0"/>
+    <visual>
+      <origin xyz="-0.12 0 ${body_z - base_z}" rpy="0 0 0"/>
       <geometry>
         <cylinder radius="${body_radius}" length="${body_height}"/>
       </geometry>
       <material name="grey"/>
-    </visual> -->
+    </visual>
     <collision>
-      <origin xyz="0 0 ${body_z - base_z}" rpy="0 0 0"/>
+      <origin xyz="-0.12 0 ${body_z - base_z}" rpy="0 0 0"/>
       <geometry>
         <cylinder radius="${body_radius}" length="${body_height}"/>
@@ -46,7 +56,7 @@
     </collision>
     <inertial>
-      <!-- Масса/инерция — грубая оценка, TO-DO -->
+      <!-- Mass and inertia are rough estimates, TO-DO -->
       <mass value="62.0"/>
-      <origin xyz="0 0 0.3" rpy="0 0 0"/>
+      <origin xyz="-0.12 0 0.3" rpy="0 0 0"/>
       <inertia ixx="5.0" ixy="0.0" ixz="0.0" iyy="5.0" iyz="0.0" izz="2.0"/>
     </inertial>
@@ -57,5 +67,5 @@
     <origin xyz="0 0 ${base_z}" rpy="0 0 0"/>
   </joint>
-  <!-- ===================== Макрос колеса ================================ -->
+  <!-- ===================== Wheel macro ================================== -->
   <xacro:macro name="wheel" params="prefix y_offset">
     <link name="${prefix}_wheel_link">
@@ -87,5 +97,40 @@
   <xacro:wheel prefix="left"  y_offset="${ wheel_separation/2}"/>
   <xacro:wheel prefix="right" y_offset="${-wheel_separation/2}"/>
-  <!-- ===================== Макрос парктроника =========================== -->
+  <!-- ===================== Caster macro (rear support) ================== -->
+  <!-- Real robot has two rear supports. Modeled as spheres:
+       fixed joint + zero friction in Gazebo (see guide_robot.gazebo.xacro).
+       Radius = base_z, center in wheel axle plane -> sphere bottom touches
+       the floor, robot rests level on 4 points. diff_drive_controller ignores
+       them (odometry uses driven wheels only). -->
+  <xacro:macro name="caster" params="prefix y_offset">
+    <link name="${prefix}_caster_link">
+      <visual>
+        <origin xyz="0 0 0" rpy="0 0 0"/>
+        <geometry>
+          <sphere radius="${caster_radius}"/>
+        </geometry>
+        <material name="dark"/>
+      </visual>
+      <collision>
+        <origin xyz="0 0 0" rpy="0 0 0"/>
+        <geometry>
+          <sphere radius="${caster_radius}"/>
+        </geometry>
+      </collision>
+      <inertial>
+        <!-- Sphere inertia: I = 2/5 * m * r^2 = 2/5 * 0.2 * 0.075^2 -->
+        <mass value="0.2"/>
+        <inertia ixx="0.00045" ixy="0" ixz="0" iyy="0.00045" iyz="0" izz="0.00045"/>
+      </inertial>
+    </link>
+    <joint name="${prefix}_caster_joint" type="fixed">
+      <parent link="base_link"/>
+      <child  link="${prefix}_caster_link"/>
+      <origin xyz="${caster_x} ${y_offset} 0" rpy="0 0 0"/>
+    </joint>
+  </xacro:macro>
+  <xacro:caster prefix="left"  y_offset="${ caster_y}"/>
+  <xacro:caster prefix="right" y_offset="${-caster_y}"/>
+  <!-- ===================== Sonar (parking sensor) macro ================= -->
   <xacro:macro name="sonar_sensor" params="id x y yaw">
     <link name="sonar_sensor_${id}"/>
@@ -96,18 +141,18 @@
     </joint>
   </xacro:macro>
-  <!-- Два спереди -->
+  <!-- Two front -->
   <xacro:sonar_sensor id="1" x="0.15"  y="0.10"  yaw="0"/>
   <xacro:sonar_sensor id="9" x="0.15"  y="-0.10" yaw="0"/>
-  <!-- Левый борт -->
+  <!-- Left side -->
   <xacro:sonar_sensor id="2" x="-0.040039" y="0.260183"  yaw="90"/>
   <xacro:sonar_sensor id="4" x="-0.393220" y="0.132040"  yaw="138.03"/>
-  <!-- Правый борт -->
+  <!-- Right side -->
   <xacro:sonar_sensor id="8" x="-0.040039" y="-0.260183" yaw="-90"/>
   <xacro:sonar_sensor id="6" x="-0.393220" y="-0.132040" yaw="-138.03"/>
-  <!-- Один сзади -->
+  <!-- One rear -->
   <xacro:sonar_sensor id="5" x="-0.435289" y="0.0"       yaw="180"/>
-  <!-- ===================== Крепления лидаров + палка ===================== -->
-  <!-- Меш lidars_mount.stl — крепёжная площадка под каждый лидар.
-       Лазерные фреймы теперь висят на этих линках, а не напрямую на base_link. -->
+  <!-- ===================== Lidar mounts + bar ========================== -->
+  <!-- lidars_mount.stl is the mounting plate under each lidar.
+       Laser frames attach to these links instead of base_link directly. -->
   <xacro:macro name="lidar_mount" params="prefix y_offset xyz_mesh:='0 0 0' rpy_mesh:='0 0 0'">
     <link name="${prefix}_lidar_mount_link">
@@ -120,5 +165,5 @@
       </visual>
       <collision>
-        <!-- Упрощённый бокс вместо полного меша — дешевле для костмапа -->
+        <!-- Simplified box instead of full mesh - cheaper for costmap -->
         <origin xyz="0 0 0.02" rpy="0 0 0"/>
         <geometry>
@@ -138,8 +183,8 @@
   </xacro:macro>
   <xacro:lidar_mount prefix="left"  y_offset="${ lidar_y_offset}"/>
-  <!-- TO-DO: правое крепление — вероятно зеркальное. Если меш в RViz "смотрит не туда",
-       крути rpy_mesh (обычно 180° по Z или по X, зависит от того как смоделирован STL). -->
+  <!-- TO-DO: right mount is probably mirrored. If the mesh faces the wrong way
+       in RViz, adjust rpy_mesh (usually 180 deg around Z or X). -->
   <xacro:lidar_mount prefix="right" y_offset="${-lidar_y_offset}" rpy_mesh="0 0 0"/>
-  <!-- Соединительный профиль между двумя креплениями -->
+  <!-- Connecting profile between the two mounts -->
   <link name="lidar_bar_link">
     <visual>
@@ -153,5 +198,5 @@
       <origin xyz="0 0 0" rpy="0 0 0"/>
       <geometry>
-        <!-- TO-DO: сверить длину/сечение с реальным bounding box 2020.stl -->
+        <!-- TO-DO: verify length and cross-section against real 2020 bounding box -->
         <box size="0.02 ${lidar_y_offset*2} 0.02"/>
       </geometry>
@@ -167,12 +212,12 @@
     <origin xyz="0.077 0.0 ${lidar_z}" rpy="0 0 0"/>
   </joint>
-  <!-- ===================== LiDAR ========================================= -->
-  <!-- Лазерные фреймы теперь на креплениях, а не на base_link.
-       z-offset 0.03 — плейсхолдер высоты корпуса лидара над плитой крепления, TO-DO уточнить. -->
+  <!-- ===================== LiDAR frames ================================ -->
+  <!-- Laser frames sit on the mounts, not on base_link.
+       z-offset 0.03 is a placeholder for lidar body height, TO-DO verify. -->
   <link name="laser_frame_left"/>
   <joint name="laser_joint_left" type="fixed">
     <parent link="left_lidar_mount_link"/>
     <child  link="laser_frame_left"/>
-    <origin xyz="0 0 0.03" rpy="0 0 0"/>
+    <origin xyz="0 0 0.03" rpy="${pi} 0 0"/>
   </joint>
   <link name="laser_frame_right"/>
@@ -180,8 +225,8 @@
     <parent link="right_lidar_mount_link"/>
     <child  link="laser_frame_right"/>
-    <origin xyz="0 0 0.03" rpy="0 0 0"/>
-  </joint>
-  <!-- ===================== IMU ========================== -->
-  <!-- TO-DO -->
+    <origin xyz="0 0 0.03" rpy="${pi} 0 0"/>
+  </joint>
+  <!-- ===================== IMU ========================================= -->
+  <!-- TO-DO: verify real IMU position -->
   <link name="imu_link"/>
   <joint name="imu_joint" type="fixed">
@@ -190,5 +235,9 @@
     <origin xyz="0 0 0.1" rpy="0 0 0"/>
   </joint>
-  <!-- ===================== ros2_control интерфейс ======================= -->
+  <!-- ===================== ros2_control interface ====================== -->
   <xacro:include filename="$(find guide_robot_description)/urdf/guide_robot.ros2_control.xacro"/>
+  <!-- ===================== Gazebo (simulation only) ==================== -->
+  <xacro:if value="$(arg use_sim)">
+    <xacro:include filename="$(find guide_robot_description)/urdf/guide_robot.gazebo.xacro"/>
+  </xacro:if>
 </robot>
