Commit message: fix(hardware): calibrate odometry, wheel separation and drive speed from measurements
ticks_per_rev was 262144 (512x8x64) assuming octal quadrature decoding;
the real decoder is x4, giving 131072. wheel_radius was the vendor's
0.075 (WheelDiameter/2), measured rolling radius is 0.1026. Together
these explain the observed 2.74x odometry undercount.

wheel_separation tape-measured at 0.347 vs vendor's 0.338 (URDF, real
geometry). In-place rotation shows an effective separation of 0.3559
for the odometry model (wide tires scrub sideways on a spin-in-place
turn), applied as wheel_separation_multiplier in the controller only -
kept separate from the geometric value used for TF.

speed_coefficient was 0.0008 m/s/unit, 5.7x off the vendor's
0.00014; measured via commanded vs actual /odom speed, corrected to
0.0001706 (now ~20% off vendor, in line with the other measured
constants).

Added linear/angular velocity and acceleration limits to
diff_drive_controller - previously unset. Deceleration is set well
above acceleration since it is the only software brake available
(cmd_vel_timeout only zeroes the commanded velocity).

All values measured on hardware (floor-rolling and spin-in-place
tests); simulation packages and temp_controllers.yaml are unaffected.

Co-Authored-By: Claude Sonnet 5 <noreply@anthropic.com>
Claude-Session: https://claude.ai/code/session_01Q1UcdBJAHSsxp365yCGMyr

File: guide_robot_description/urdf/guide_robot.ros2_control.xacro (robot description, xacro)
@@ -31,10 +31,10 @@
           <param name="left_wheel_id">46</param>                 <!-- 0x2E -->
           <param name="right_wheel_id">47</param>                <!-- 0x2F -->
-          <param name="ticks_per_rev">262144</param>             <!-- 512*8*64 -->
+          <param name="ticks_per_rev">131072</param>             <!-- 512*4*64, quadrature is x4 not x8 (measured) -->
           <param name="left_sign">1</param>
           <param name="right_sign">-1</param>                    <!-- right wheel inverted physically -->
           <param name="swap_drives">1</param>                    <!-- FURO_SWAP_DRIVES -->
-          <param name="speed_coefficient">0.0008</param>         <!-- m/s per motor unit -->
-          <param name="wheel_radius">0.075</param>               <!-- wheel radius in meters -->
+          <param name="speed_coefficient">0.0001706</param>      <!-- m/s per motor unit, measured (2026-07-26): cmd 0.2 m/s -> odom avg 0.0426 m/s over 3 runs -->
+          <param name="wheel_radius">0.1026</param>              <!-- rolling radius, measured: 3.157 m over 30.758 rad -->
           <param name="cmd_timeout">0.3</param>                  <!-- watchdog, seconds -->
         </xacro:unless>

File: guide_robot_description/urdf/guide_robot.urdf.xacro (robot description, xacro)
@@ -14,6 +14,10 @@
   <xacro:arg name="use_sim" default="false"/>
   <!-- ===================== Parameters (from robot_params.yaml) =========== -->
-  <xacro:property name="wheel_separation" value="0.338"/>   <!-- WheelBase -->
-  <xacro:property name="wheel_radius"     value="0.075"/>    <!-- WheelDiameter/2 -->
+  <!-- Geometric track width, tape-measured wheel centerline to centerline
+       (RobotSetting.xml said 0.338 - wrong, like the wheel diameter).
+       The controller uses a slightly larger EFFECTIVE value, see
+       guide_robot_controllers.yaml - do not sync the two numbers. -->
+  <xacro:property name="wheel_separation" value="0.347"/>
+  <xacro:property name="wheel_radius"     value="0.1026"/>   <!-- rolling radius, measured (RobotSetting.xml said 0.075 - wrong) -->
   <xacro:property name="wheel_width"      value="0.048"/>    <!-- WheelWidth -->
   <!-- Body dimensions - rough estimate of top-heavy chassis -->
@@ -119,7 +123,7 @@
       </collision>
       <inertial>
-        <!-- Sphere inertia: I = 2/5 * m * r^2 = 2/5 * 0.2 * 0.075^2 -->
+        <!-- Sphere inertia: I = 2/5 * m * r^2 = 2/5 * 0.2 * 0.1026^2 -->
         <mass value="0.2"/>
-        <inertia ixx="0.00045" ixy="0" ixz="0" iyy="0.00045" iyz="0" izz="0.00045"/>
+        <inertia ixx="0.00084" ixy="0" ixz="0" iyy="0.00084" iyz="0" izz="0.00084"/>
       </inertial>
     </link>
