Commit message: feat: add fully working sim and sonars

File: guide_robot_description/urdf/guide_robot.gazebo.xacro (robot description, xacro)
@@ -142,5 +142,59 @@
     <mu2>0.0</mu2>
   </gazebo>
-  <!-- TO-DO: 7 sonars as Gazebo ray sensors -> guide_robot_msgs/SonarRanges.
-       Skipped for now: /scan alone is enough for the Nav2 baseline. -->
+  <!-- ===================================================================== -->
+  <!--  5. Sonars (parking sensors) -> /sonar/raw/sonar_<id> (sensor_msgs/Range)   -->
+  <!--     Aggregated into guide_robot_msgs/SonarRanges by sonar_aggregator. -->
+  <!--     Typical automotive parking sensor: ~40 kHz, 0.2..2.5 m, cone 30 deg -->
+  <!-- ===================================================================== -->
+  <xacro:macro name="sonar_gazebo" params="id">
+    <gazebo reference="sonar_sensor_${id}">
+      <sensor type="ray" name="sonar_${id}">
+        <pose>0 0 0 0 0 0</pose>
+        <visualize>true</visualize>
+        <update_rate>10</update_rate>
+        <ray>
+          <scan>
+            <horizontal>
+              <samples>7</samples>
+              <resolution>1</resolution>
+              <min_angle>-0.52</min_angle>   <!-- +-30 deg = 60 deg cone -->
+              <max_angle> 0.52</max_angle>
+            </horizontal>
+            <vertical>
+              <samples>5</samples>
+              <resolution>1</resolution>
+              <min_angle>-0.26</min_angle>
+              <max_angle> 0.26</max_angle>
+            </vertical>
+          </scan>
+          <range>
+            <min>0.20</min>
+            <max>2.50</max>
+            <resolution>0.01</resolution>
+          </range>
+          <noise>
+            <type>gaussian</type>
+            <mean>0.0</mean>
+            <stddev>0.01</stddev>
+          </noise>
+        </ray>
+        <plugin name="sonar_${id}_controller" filename="libgazebo_ros_ray_sensor.so">
+          <ros>
+            <remapping>~/out:=sonar/raw/sonar_${id}</remapping>
+          </ros>
+          <!-- Range output takes the MINIMUM over all rays in the cone -->
+          <output_type>sensor_msgs/Range</output_type>
+          <radiation_type>ultrasound</radiation_type>
+          <frame_name>sonar_sensor_${id}</frame_name>
+        </plugin>
+      </sensor>
+    </gazebo>
+  </xacro:macro>
+  <xacro:sonar_gazebo id="1"/>
+  <xacro:sonar_gazebo id="2"/>
+  <xacro:sonar_gazebo id="4"/>
+  <xacro:sonar_gazebo id="5"/>
+  <xacro:sonar_gazebo id="6"/>
+  <xacro:sonar_gazebo id="8"/>
+  <xacro:sonar_gazebo id="9"/>
 </robot>

File: guide_robot_description/urdf/guide_robot.urdf.xacro (robot description, xacro)
@@ -134,11 +134,20 @@
   <!-- ===================== Sonar (parking sensor) macro ================= -->
   <xacro:macro name="sonar_sensor" params="id x y yaw">
-    <link name="sonar_sensor_${id}"/>
-    <joint name="sonar_sensor_${id}_joint" type="fixed">
-      <parent link="base_link"/>
-      <child  link="sonar_sensor_${id}"/>
-      <origin xyz="${x} ${y} 0.2" rpy="0 0 ${radians(yaw)}"/>
-    </joint>
-  </xacro:macro>
+      <link name="sonar_sensor_${id}">
+        <visual>
+          <geometry><box size="0.01 0.02 0.01"/></geometry>
+          <material name="dark"/>
+        </visual>
+        <inertial>
+          <mass value="0.01"/>
+          <inertia ixx="1e-6" ixy="0" ixz="0" iyy="1e-6" iyz="0" izz="1e-6"/>
+        </inertial>
+      </link>
+      <joint name="sonar_sensor_${id}_joint" type="fixed">
+        <parent link="base_link"/>
+        <child  link="sonar_sensor_${id}"/>
+        <origin xyz="${x} ${y} 0.2" rpy="0 0 ${radians(yaw)}"/>
+      </joint>
+    </xacro:macro>
   <!-- Two front -->
   <xacro:sonar_sensor id="1" x="0.15"  y="0.10"  yaw="0"/>

Commit message: feat: add correct robot_params.yaml parsers

File: guide_robot_description/urdf/guide_robot.gazebo.xacro (robot description, xacro)
@@ -17,7 +17,9 @@
   <!--     URDF from robot_state_publisher breaks the CLI param parser.        -->
   <!-- ===================================================================== -->
-<gazebo>
+  <xacro:arg name="controllers_file"
+           default="$(find guide_robot_description)/config/controllers.yaml"/>
+  <gazebo>
     <plugin filename="libgazebo_ros2_control.so" name="gazebo_ros2_control">
-      <parameters>$(find guide_robot_description)/params/temp_controllers.yaml</parameters>
+      <parameters>$(arg controllers_file)</parameters>
     </plugin>
   </gazebo>

File: guide_robot_description/urdf/guide_robot.ros2_control.xacro (robot description, xacro)
@@ -6,4 +6,7 @@
        use_mock_hardware=true -> mock_components stub for stack testing
        otherwise              -> real Dynamixel base driver (FURO)
+     NOT standalone-processable: relies on properties declared by
+     guide_robot.urdf.xacro before the include point - p, wheel_separation,
+     wheel_radius. Process the main xacro, not this file.
      IMPORTANT: comments MUST stay ASCII-only (see note in guide_robot.urdf.xacro).
      ========================================================================= -->
@@ -11,4 +14,27 @@
   <xacro:arg name="use_sim"           default="false"/>
   <xacro:arg name="use_mock_hardware" default="false"/>
+  <xacro:property name="lim" value="${p['limits']}"/>
+  <xacro:property name="drv" value="${p['drive']}"/>
+  <!-- Per-wheel command envelope. Worst case is full linear PLUS full angular
+       applied at once:
+         v_wheel = v_max + w_max * wheel_separation / 2
+         w_wheel = v_wheel / wheel_radius * wheel_limit_margin
+       With the current robot_params.yaml this evaluates to 8.38 rad/s.
+       This is an ENVELOPE, not a limit: actual clamping is done by
+       diff_drive_controller. Too narrow drops commands, too wide is harmless,
+       hence the margin. Recomputed automatically - do not hardcode. -->
+  <xacro:property name="w_wheel_max"
+    value="${((lim['max_linear_velocity'] + lim['max_angular_velocity']*wheel_separation/2)
+              / wheel_radius * lim['wheel_limit_margin'])}"/>
+  <xacro:macro name="wheel_iface" params="name">
+    <joint name="${name}">
+      <command_interface name="velocity">
+        <param name="min">${-w_wheel_max}</param>   <!-- rad/s -->
+        <param name="max">${w_wheel_max}</param>
+      </command_interface>
+      <state_interface name="position"/>
+      <state_interface name="velocity"/>
+    </joint>
+  </xacro:macro>
   <ros2_control name="GuideRobotSystem" type="system">
     <hardware>
@@ -25,47 +51,24 @@
         </xacro:if>
         <xacro:unless value="$(arg use_mock_hardware)">
-          <!-- Real FURO Dynamixel base driver. -->
+          <!-- Real FURO Dynamixel base driver. All values come from
+               config/robot_params.yaml, section 'drive' - see that file for
+               measurement provenance. -->
           <plugin>guide_robot_hardware/GuideRobotSystem</plugin>
-          <param name="serial_port">/dev/tty_motors</param>      <!-- udev symlink, see scripts/99-furo-devices.rules -->
-          <param name="baud_rate">115200</param>
-          <param name="left_wheel_id">46</param>                 <!-- 0x2E -->
-          <param name="right_wheel_id">47</param>                <!-- 0x2F -->
-          <param name="ticks_per_rev">131072</param>             <!-- 512*4*64, quadrature is x4 not x8 (measured) -->
-          <param name="left_sign">1</param>
-          <param name="right_sign">-1</param>                    <!-- right wheel inverted physically -->
-          <param name="swap_drives">1</param>                    <!-- FURO_SWAP_DRIVES -->
-          <param name="speed_coefficient">0.0001706</param>      <!-- m/s per motor unit, measured (2026-07-26): cmd 0.2 m/s -> odom avg 0.0426 m/s over 3 runs -->
-          <param name="wheel_radius">0.1026</param>              <!-- rolling radius, measured: 3.157 m over 30.758 rad -->
-          <param name="cmd_timeout">0.3</param>                  <!-- watchdog, seconds -->
+          <param name="serial_port">${drv['serial_port']}</param>
+          <param name="baud_rate">${drv['baud_rate']}</param>
+          <param name="left_wheel_id">${drv['left_wheel_id']}</param>
+          <param name="right_wheel_id">${drv['right_wheel_id']}</param>
+          <param name="ticks_per_rev">${drv['ticks_per_rev']}</param>
+          <param name="left_sign">${drv['left_sign']}</param>
+          <param name="right_sign">${drv['right_sign']}</param>
+          <param name="swap_drives">${drv['swap_drives']}</param>
+          <param name="speed_coefficient">${drv['speed_coefficient']}</param>
+          <param name="wheel_radius">${wheel_radius}</param>
+          <param name="cmd_timeout">${drv['cmd_timeout']}</param>
         </xacro:unless>
       </xacro:unless>
     </hardware>
-    <!-- Per-wheel envelope must cover the WORST CASE of the base limits in
-         guide_robot_controllers.yaml, which is full linear PLUS full angular:
-           v_wheel = v_max + w_max * wheel_separation_eff / 2
-                   = 0.6 + 1.0472 * 0.35597 / 2 = 0.7864 m/s
-           w_wheel = 0.7864 / 0.1026 = 7.66 rad/s
-         The old 6.98 was below that after the 2026-07-27 speed doubling, so a
-         simultaneous drive+turn at full command would have sat outside the
-         declared range. Raised to 8.0 rad/s (0.82 m/s) to keep margin.
-         Recompute this whenever the yaml limits or wheel_radius change. -->
-    <!-- Left wheel -->
-    <joint name="left_wheel_joint">
-      <command_interface name="velocity">
-        <param name="min">-8.0</param>   <!-- rad/s -->
-        <param name="max">8.0</param>
-      </command_interface>
-      <state_interface name="position"/>
-      <state_interface name="velocity"/>
-    </joint>
-    <!-- Right wheel -->
-    <joint name="right_wheel_joint">
-      <command_interface name="velocity">
-        <param name="min">-8.0</param>
-        <param name="max">8.0</param>
-      </command_interface>
-      <state_interface name="position"/>
-      <state_interface name="velocity"/>
-    </joint>
+    <xacro:wheel_iface name="left_wheel_joint"/>
+    <xacro:wheel_iface name="right_wheel_joint"/>
   </ros2_control>
 </robot>

File: guide_robot_description/urdf/guide_robot.urdf.xacro (robot description, xacro)
@@ -14,33 +14,25 @@
   <xacro:arg name="use_sim" default="false"/>
   <!-- ===================== Parameters (from robot_params.yaml) =========== -->
-  <!-- Geometric track width, tape-measured wheel centerline to centerline
-       (RobotSetting.xml said 0.338 - wrong, like the wheel diameter).
-       The controller uses a slightly larger EFFECTIVE value, see
-       guide_robot_controllers.yaml - do not sync the two numbers. -->
-  <xacro:property name="wheel_separation" value="0.347"/>
-  <xacro:property name="wheel_radius"     value="0.1026"/>   <!-- rolling radius, measured (RobotSetting.xml said 0.075 - wrong) -->
-  <xacro:property name="wheel_width"      value="0.048"/>    <!-- WheelWidth -->
-  <!-- Body dimensions - rough estimate of top-heavy chassis -->
-  <xacro:property name="body_radius" value="0.31"/>
-  <xacro:property name="body_height" value="1.62"/>
-  <xacro:property name="body_z"      value="0.885"/>         <!-- body center Z -->
-  <!-- Ground clearance: wheel axle height above floor = wheel_radius -->
-  <xacro:property name="base_z" value="${wheel_radius}"/>
-  <!-- Rear casters (real support) -->
-  <xacro:property name="caster_radius" value="${base_z}"/>   <!-- = wheel_radius, keeps robot level -->
-  <xacro:property name="caster_x"      value="-0.3"/>       <!-- behind base center, ~20 cm -->
-  <xacro:property name="caster_y"      value="0.12"/>        <!-- lateral spacing -->
+  <xacro:property name="params_file"
+                  value="$(find guide_robot_description)/config/robot_params.yaml"/>
+  <xacro:property name="p" value="${xacro.load_yaml(params_file)}"/>
+  <xacro:property name="g" value="${p['geometry']}"/>
+  <xacro:property name="wheel_separation" value="${g['wheel_separation']}"/>
+  <xacro:property name="wheel_radius"     value="${g['wheel_radius']}"/>
+  <xacro:property name="wheel_width"      value="${g['wheel_width']}"/>
+  <xacro:property name="body_radius"      value="${g['body_radius']}"/>
+  <xacro:property name="body_height"      value="${g['body_height']}"/>
+  <xacro:property name="body_z"           value="${g['body_z']}"/>
+  <xacro:property name="caster_x"         value="${g['caster_x']}"/>
+  <xacro:property name="caster_y"         value="${g['caster_y']}"/>
+  <xacro:property name="lidar_x_offset"   value="${g['lidar_x_offset']}"/>
+  <xacro:property name="lidar_y_offset"   value="${g['lidar_y_offset']}"/>
+  <xacro:property name="lidar_z"          value="${g['lidar_z']}"/>
+  <xacro:property name="base_z"           value="${wheel_radius}"/>
+  <xacro:property name="caster_radius"    value="${wheel_radius}"/>
   <!-- Lidar mounts + connecting bar (2020 extrusion) -->
   <xacro:property name="lidar_mount_mesh" value="package://guide_robot_description/meshes/lidars_mount.stl"/>
   <xacro:property name="lidar_bar_mesh"   value="package://guide_robot_description/meshes/al_profile.stl"/>
-  <!-- TO-DO: if meshes were exported from CAD in mm, scale 0.001 is required.
-       Check in RViz: huge or tiny model means wrong scale. -->
   <xacro:property name="mesh_scale" value="0.001 0.001 0.001"/>
-  <xacro:property name="lidar_y_offset" value="0.258"/>      <!-- from laser_joint_left/right -->
-  <!-- Measured floor->lidar height 0.495 m; lidar_z = 0.495 - base_z - 0.03 -->
-  <xacro:property name="lidar_z" value="0.3624"/>
-  <!-- Measured: wheel/floor point to wall 0.363 m, lidar to wall 0.283 m;
-       lidar_x_offset = 0.363 - 0.283 -->
-  <xacro:property name="lidar_x_offset" value="0.08"/>
   <!-- ===================== RViz materials =============================== -->
   <material name="grey"><color rgba="0.4 0.4 0.45 1.0"/></material>
