Commit message: fix(description): correct lidar frame orientation to match the real mount
Оба лидара стоят перевёрнутыми и развёрнутыми «нос-хвост». Поворот
вокруг pitch (а не roll) переворачивает X (вперёд->назад) и Z (верх/низ),
оставляя Y нетронутым — именно это отправляет луч с сырым углом 0,
который смотрел вперёд, назад, как на реальном креплении.

Для симуляции это чистая смена конвенции: gazebo_ros_ray_sensor привязан
к тем же laser_frame_left/right (guide_robot.gazebo.xacro) и публикует
с тем же frame_id, поэтому данные и TF остаются согласованными.

Co-Authored-By: Claude Opus 5 <noreply@anthropic.com>
Claude-Session: https://claude.ai/code/session_0177m9aCApSnSvTvQRvDJ7s3

File: guide_robot_description/urdf/guide_robot.urdf.xacro (robot description, xacro)
@@ -223,10 +223,15 @@
   <!-- ===================== LiDAR frames ================================ -->
   <!-- Laser frames sit on the mounts, not on base_link.
-       z-offset 0.03 is a placeholder for lidar body height, TO-DO verify. -->
+       z-offset 0.03 is a placeholder for lidar body height, TO-DO verify.
+       Both lidars are physically mounted upside-down AND front-to-back
+       reversed. Rotating about pitch (not roll) flips X (forward->backward)
+       and Z (up/down), while leaving Y (left/right) untouched - this is
+       what makes the raw angle-0 ray, which pointed toward robot-forward,
+       point toward robot-backward instead, matching the real mount. -->
   <link name="laser_frame_left"/>
   <joint name="laser_joint_left" type="fixed">
     <parent link="left_lidar_mount_link"/>
     <child  link="laser_frame_left"/>
-    <origin xyz="0 0 0.03" rpy="${pi} 0 0"/>
+    <origin xyz="0 0 0.03" rpy="0 ${pi} 0"/>
   </joint>
   <link name="laser_frame_right"/>
@@ -234,5 +239,5 @@
     <parent link="right_lidar_mount_link"/>
     <child  link="laser_frame_right"/>
-    <origin xyz="0 0 0.03" rpy="${pi} 0 0"/>
+    <origin xyz="0 0 0.03" rpy="0 ${pi} 0"/>
   </joint>
   <!-- ===================== IMU ========================================= -->

Commit message: fix(description): calibrate lidar X/Z offsets from tape measurements
lidar_x_offset and lidar_z were unverified placeholders (0.075/0.077,
0.4). Measured directly on hardware: wheel/floor point to wall 0.363 m,
lidar's own optical center to the same wall 0.283 m -> x = 0.08 m.
Floor to lidar height 0.495 m, minus base_z and the fixed 0.03 mount
standoff -> lidar_z = 0.3624 m.

Co-Authored-By: Claude Sonnet 5 <noreply@anthropic.com>
Claude-Session: https://claude.ai/code/session_01Q1UcdBJAHSsxp365yCGMyr

File: guide_robot_description/urdf/guide_robot.urdf.xacro (robot description, xacro)
@@ -38,5 +38,9 @@
   <xacro:property name="mesh_scale" value="0.001 0.001 0.001"/>
   <xacro:property name="lidar_y_offset" value="0.258"/>      <!-- from laser_joint_left/right -->
-  <xacro:property name="lidar_z" value="0.4"/>
+  <!-- Measured floor->lidar height 0.495 m; lidar_z = 0.495 - base_z - 0.03 -->
+  <xacro:property name="lidar_z" value="0.3624"/>
+  <!-- Measured: wheel/floor point to wall 0.363 m, lidar to wall 0.283 m;
+       lidar_x_offset = 0.363 - 0.283 -->
+  <xacro:property name="lidar_x_offset" value="0.08"/>
   <!-- ===================== RViz materials =============================== -->
   <material name="grey"><color rgba="0.4 0.4 0.45 1.0"/></material>
@@ -192,5 +196,5 @@
       <parent link="base_link"/>
       <child  link="${prefix}_lidar_mount_link"/>
-      <origin xyz="0.075 ${y_offset} ${lidar_z}" rpy="0 0 0"/>
+      <origin xyz="${lidar_x_offset} ${y_offset} ${lidar_z}" rpy="0 0 0"/>
     </joint>
   </xacro:macro>
@@ -223,5 +227,5 @@
     <parent link="base_link"/>
     <child  link="lidar_bar_link"/>
-    <origin xyz="0.077 0.0 ${lidar_z}" rpy="0 0 0"/>
+    <origin xyz="${lidar_x_offset} 0.0 ${lidar_z}" rpy="0 0 0"/>
   </joint>
   <!-- ===================== LiDAR frames ================================ -->

Commit message: fix(nav): rear-only drive after lidar yaw twist, plus rear sonar stop
Lidars were rotated ±90° on the mast; DWB/smoother only command −X so the
screen still faces the goal, and collision_monitor covers the new rear
travel direction.

Co-authored-by: Cursor <cursoragent@cursor.com>

File: guide_robot_description/urdf/guide_robot.urdf.xacro (robot description, xacro)
@@ -29,4 +29,6 @@
   <xacro:property name="lidar_y_offset"   value="${g['lidar_y_offset']}"/>
   <xacro:property name="lidar_z"          value="${g['lidar_z']}"/>
+  <xacro:property name="lidar_left_yaw"   value="${g['lidar_left_yaw']}"/>
+  <xacro:property name="lidar_right_yaw"  value="${g['lidar_right_yaw']}"/>
   <xacro:property name="body_x_offset"    value="${g['body_x_offset']}"/>
   <xacro:property name="sonar_z"          value="${g['sonar_z']}"/>
@@ -226,14 +228,11 @@
   <!-- Laser frames sit on the mounts, not on base_link.
        z-offset 0.03 is a placeholder for lidar body height, TO-DO verify.
-       Both lidars are physically mounted upside-down AND front-to-back
-       reversed. Rotating about pitch (not roll) flips X (forward->backward)
-       and Z (up/down), while leaving Y (left/right) untouched - this is
-       what makes the raw angle-0 ray, which pointed toward robot-forward,
-       point toward robot-backward instead, matching the real mount. -->
+       Both lidars are upside-down (pitch pi). Extra yaw is the 2026-08-30
+       twist: left +90 deg CCW, right -90 deg CW, top view. -->
   <link name="laser_frame_left"/>
   <joint name="laser_joint_left" type="fixed">
     <parent link="left_lidar_mount_link"/>
     <child  link="laser_frame_left"/>
-    <origin xyz="0 0 0.03" rpy="0 ${pi} 0"/>
+    <origin xyz="0 0 0.03" rpy="0 ${pi} ${lidar_left_yaw}"/>
   </joint>
   <link name="laser_frame_right"/>
@@ -241,5 +240,5 @@
     <parent link="right_lidar_mount_link"/>
     <child  link="laser_frame_right"/>
-    <origin xyz="0 0 0.03" rpy="0 ${pi} 0"/>
+    <origin xyz="0 0 0.03" rpy="0 ${pi} ${lidar_right_yaw}"/>
   </joint>
   <!-- ===================== IMU ========================================= -->

Commit message: fix: drive caster-first via URDF yaw π and prefer +vx in DWB
Nav2 treated reverse as cruise and crept forward on 180° goals.
Flip footprint so +X is travel, keep a short −vx window for parking,
and shrink the screen-side slow polygon.

Co-authored-by: Cursor <cursoragent@cursor.com>

File: guide_robot_description/urdf/guide_robot.urdf.xacro (robot description, xacro)
@@ -69,5 +69,8 @@
     <parent link="base_footprint"/>
     <child  link="base_link"/>
-    <origin xyz="0 0 ${base_z}" rpy="0 0 0"/>
+    <!-- +X footprint = casters (travel). base_link (screen, old +X) is yaw pi
+         so Nav2 uses +vx. Hardware: both signs flipped and swap_drives 0,
+         otherwise wz reverses with vx. -->
+    <origin xyz="0 0 ${base_z}" rpy="0 0 ${pi}"/>
   </joint>
   <!-- ===================== Wheel macro ================================== -->

Commit message: fix(sim): match Gazebo wheel joints to the caster-first URDF yaw pi
592c93f flipped the robot's travel direction by yaw-pi-ing base_link
inside base_footprint_joint, compensating on hardware with inverted
left_sign/right_sign and swap_drives 0 in guide_robot_hardware. That
compensation only exists for the real FURO driver: gazebo_ros2_control's
GazeboSystem has no equivalent knob, so the wheel joints (still defined
in base_link, unchanged axis/offset) ended up geometrically flipped
relative to base_footprint - left and right swapped, axis pointing -Y.
diff_drive_controller commands were consequently correct in wz but
inverted in vx: the sim drove backwards from what /cmd_vel asked for.

Negate wheel joint origin/axis in the wheel macro so left_wheel_joint/
right_wheel_joint are geometrically canonical in base_footprint again.
This is unconditional (not use_sim-only): the real hardware driver
addresses wheels by joint name and reads drive signs from
robot_params.yaml params, never from URDF geometry, so the only effect
there is fixing wheels that currently spin backwards in RViz.

Also add a spawn_yaw launch arg (default pi) to gazebo.launch.py,
plumbed through simulation.launch.py, since spawn_entity had no -Y and
was spawning the robot at yaw 0 while AMCL's initial_pose.yaw is pi
with recovery_alpha_* disabled - a guaranteed 180 degree localization
mismatch at startup.

Verified via `xacro ... | gz sdf -p`: left_wheel_joint now lands at
y=+0.1735 in base_footprint (was -0.1735), matching the diff-drive
canon.

Co-Authored-By: Claude Opus 5 (1M context) <noreply@anthropic.com>
Claude-Session: https://claude.ai/code/session_01JBvdrcC4uRsq971HHSkDn5

File: guide_robot_description/urdf/guide_robot.urdf.xacro (robot description, xacro)
@@ -71,5 +71,7 @@
     <!-- +X footprint = casters (travel). base_link (screen, old +X) is yaw pi
          so Nav2 uses +vx. Hardware: both signs flipped and swap_drives 0,
-         otherwise wz reverses with vx. -->
+         otherwise wz reverses with vx. Wheel joints below negate origin and
+         axis to compensate this same yaw pi for Gazebo, which has no
+         left_sign/right_sign/swap_drives equivalent. -->
     <origin xyz="0 0 ${base_z}" rpy="0 0 ${pi}"/>
   </joint>
@@ -98,6 +100,11 @@
       <parent link="base_link"/>
       <child  link="${prefix}_wheel_link"/>
-      <origin xyz="0 ${y_offset} 0" rpy="0 0 0"/>
-      <axis xyz="0 1 0"/>
+      <!-- Joint origin and axis are in base_link, which base_footprint_joint
+           turns by yaw pi. Both are negated so that in base_footprint the
+           result is the diff-drive canon: left at +b/2 with axis +Y. Without
+           this the sim drives -vx - GazeboSystem has no left_sign/right_sign/
+           swap_drives to flip it (see base_footprint_joint above). -->
+      <origin xyz="0 ${-y_offset} 0" rpy="0 0 0"/>
+      <axis xyz="0 -1 0"/>
     </joint>
   </xacro:macro>
